Commit message: Fix controller fighting issue

File: mirte_description/mirte_master_description/urdf/lidar.xacro (robot description, xacro)
@@ -95,9 +95,11 @@
               <frame_name>lidar_link</frame_name>
               <topic_name>scan</topic_name>
-              <yaw_correction>0</yaw_correction>
               <ego_filter>
                 <enabled>true</enabled>
                 <min_range>0.01</min_range>
-                <footprint>-0.096 -0.069, -0.096 0.069, 0.02 0.069, 0.02 -0.069</footprint>
+                <footprint>0.0283 0.1021, 0.0283 0.1384, 0.0715 0.1384, 0.0715 0.1021</footprint>
+                <footprint_0>-0.1034 -0.0732, -0.1034 -0.0343, -0.0677 -0.0343, -0.0677 -0.0732</footprint_0>
+                <footprint_1>0.0991 -0.0202, 0.0991 0.0245, 0.1358 0.0245, 0.1358 -0.0202</footprint_1>
+                <footprint_2>-0.1034 0.0343, -0.1034 0.0732, -0.0677 0.0732, -0.0677 0.0343</footprint_2>
               </ego_filter>
             </plugin>

File: mirte_description/mirte_master_description/urdf/ros2_control.xacro (robot description, xacro)
@@ -49,5 +49,5 @@
         <command_interface name="position"/>
         <state_interface name="position">
-          <param name="initial_value">-1.56</param>
+          <!-- <param name="initial_value">-1.56</param> -->
         </state_interface>
         <state_interface name="velocity" />
@@ -56,5 +56,5 @@
         <command_interface name="position"/>
         <state_interface name="position">
-          <param name="initial_value">-1.56</param>
+          <!-- <param name="initial_value">-1.56</param> -->
         </state_interface>
         <state_interface name="velocity" />
@@ -63,5 +63,5 @@
         <command_interface name="position"/>
         <state_interface name="position">
-          <param name="initial_value">1.56</param>
+          <!-- <param name="initial_value">1.56</param> -->
         </state_interface>
         <state_interface name="velocity" />

File: mirte_description/mirte_master_description/urdf/wheel.xacro (robot description, xacro)
@@ -38,4 +38,5 @@
     <child link="${name}_wheel" />
     <axis xyz="0 0 -1" />
+    <dynamics damping="0.05" friction="0.0"/>
   </joint>
   <transmission name="${name}_wheel_transmission">
